File: 05_硬件研发/原理图/KiCad/EL-1000_PowerStage.kicad_sch (KiCad schematic)
At the start: 30 parts, among them Q1 M90N20, Q10 M90N20, Q11 M90N20, Q12 M90N20, Q2 M90N20, Q3 M90N20, Q4 M90N20, Q5 M90N20, Q6 M90N20, Q7 M90N20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

Commit message: 功率级原理图: 加连线和网络标号
- 53个元件 + 30条连线 + 5个net label + 5个章节标注
- HRPWM RC滤波→分压→MOSFET栅极总线
- Group A(130) / Group B(88) 栅极驱动总线
- LOAD+ 漏极公共节点
- kicad-cli验证通过
Parts:
- removed Q1, Q10, Q11, Q12, Q2, Q3, Q4, Q5, Q6, Q7, Q8, Q9: M90N20, symbol Transistor_FET:BSS138
- removed RS1, RS10, RS11, RS12, RS2, RS3, RS4, RS5, RS6, RS7, RS8, RS9: 0.05R, symbol Device:R
Other:
- note added: "=== HRPWM RC FILTER (15.2-bit) ==="
- note added: "=== MOSFET GROUP A (Q1-Q6) ==="
- note added: "=== MOSFET GROUP B (Q7-Q12) ==="
- note added: "=== PUSH-PULL DRIVER ==="
- note added: "=== VOLTAGE DIVIDER 1:13.2 ==="
- note removed: "Channel 1-6: M90N20 + 0.05R Source"
- note removed: "Channel 7-12: M90N20 + 0.05R Source"
- note removed: "EL-1000 Power Stage v0.4 — 12xM90N20 + RS6332 + MCSF2512DR050Q9"
- note removed: "HRPWM RC Filter (R1=10k, C1=1uF)"
- note removed: "Push-Pull Driver (D882/B772)"
- note removed: "Voltage Divider 1:13.2 (R2=95k, R3=5.23k)"

Commit message: 功率级原理图完成: 精确引脚连接+反馈回路
- 51个元件精确放置, 56条走线按实际引脚连接
- 信号流: HRPWM→RC滤波→分压→RS6332→推挽→MOSFET栅极
- RS6332闭环: V_REF→IN+, SUM_NODE→IN-, OUT→推挽
- VCC→+5V, VEE→GND
- 12× M90N20两组, 每管独立源极电阻
- 6个net label + 7个章节标注
- kicad-cli验证通过
Parts:
- added Q1, Q10, Q11, Q12, Q2, Q3, Q4, Q5, Q6, Q7, Q8, Q9: M90N20, symbol Transistor_FET:BSS138
- added RS1, RS10, RS11, RS12, RS2, RS3, RS4, RS5, RS6, RS7, RS8, RS9: 0.05R, symbol Device:R
- added U1 (x2): RS6332, symbol Amplifier_Operational:LM2904
Other:
- note added: "EL-1000 Power Stage v0.4"
- note added: "MOSFET Bank A - Q1..Q6"
- note added: "MOSFET Bank B - Q7..Q12"
- note added: "SECTION 1: HRPWM RC Low-Pass Filter"
- note added: "SECTION 2: Voltage Divider 1:19.2"
- note added: "SECTION 3: RS6332 Op-Amp Error Amplifier"
- note added: "SECTION 4: Push-Pull Gate Driver (D882/B772)"
- note removed: "=== HRPWM RC FILTER (15.2-bit) ==="
- note removed: "=== MOSFET GROUP A (Q1-Q6) ==="
- note removed: "=== MOSFET GROUP B (Q7-Q12) ==="
- note removed: "=== PUSH-PULL DRIVER ==="
- note removed: "=== VOLTAGE DIVIDER 1:13.2 ==="
- title: EL-1000 Power Stage v0.4 -> (none)
